File: stm32f4_uno_ethernet.kicad_pcb (KiCad board)
At the start: 2 copper layers, 68.6 x 53.3 mm, 55 parts, among them J104 STM32 GPIO, J106 Power, J107 Ethernet, J110 Analog, J111 Conn_01x04, J201 RJ45-TH_B-1-1, U201 SRV05-4, U202 LAN8742A, Y201 25MHz

Commit message: #4 Wrong polarity on C207
Parts:
- turned C207 to 180 degrees
Connections:
- C207 pad 1: GND -> /Ethernet/VDDxA
- C207 pad 2: /Ethernet/VDDxA -> GND
- J106 pad 2: unconnected-(J106-Pin_2-Pad2) -> +3V3
Routing:
- net +3V3: track 53.0 -> 60.8 mm
- net /Ethernet/VDDxA: track 78.7 -> 81.2 mm
